Commit message: update wheels

File: my_robot_description/urdf/wheels.xacro (robot description, xacro)
@@ -17,5 +17,5 @@
     <link name="${name}">
       <visual>
-        <origin xyz="0 0 0" rpy="1.57079632679 0 0"/>
+        <origin xyz="0 0 0" rpy="0 0 0"/>
         <geometry>
           <cylinder radius="${radius}" length="${width}"/>
@@ -24,5 +24,5 @@
       </visual>
       <collision>
-        <origin xyz="0 0 0" rpy="1.57079632679 0 0"/>
+        <origin xyz="0 0 0" rpy="0 0 0"/>
         <geometry>
           <cylinder radius="${radius}" length="${width}"/>
@@ -38,7 +38,7 @@
       <parent link="${parent}"/>
       <child link="${name}"/>
-      <origin xyz="${x} ${y} ${z}" rpy="0 0 0"/>
-      <!-- wheel rolls around Y (left axis), with ROS convention x forward, y left, z up -->
-      <axis xyz="0 1 0"/>
+      <origin xyz="${x} ${y} ${z}" rpy="-1.57079632679 0 0"/>
+      <!-- Keep cylinder along link-Z and rotate the joint frame so wheel axle aligns with parent Y. -->
+      <axis xyz="0 0 1"/>
     </joint>
   </xacro:macro>

Commit message: Fix wheel joint axis alignment in custom robot xacro

File: my_robot_description/urdf/wheels.xacro (robot description, xacro)
@@ -38,7 +38,7 @@
       <parent link="${parent}"/>
       <child link="${name}"/>
-      <origin xyz="${x} ${y} ${z}" rpy="-1.57079632679 0 0"/>
-      <!-- Keep cylinder along link-Z and rotate the joint frame so wheel axle aligns with parent Y. -->
-      <axis xyz="0 0 1"/>
+      <origin xyz="${x} ${y} ${z}" rpy="0 0 0"/>
+      <!-- Keep wheel link aligned with parent; set wheel axle directly on parent Y. -->
+      <axis xyz="0 1 0"/>
     </joint>
   </xacro:macro>

Commit message: update wheels

File: my_robot_description/urdf/wheels.xacro (robot description, xacro)
@@ -17,5 +17,5 @@
     <link name="${name}">
       <visual>
-        <origin xyz="0 0 0" rpy="0 0 0"/>
+        <origin xyz="0 0 0" rpy="1.57079632679 0 0"/>
         <geometry>
           <cylinder radius="${radius}" length="${width}"/>
@@ -24,5 +24,5 @@
       </visual>
       <collision>
-        <origin xyz="0 0 0" rpy="0 0 0"/>
+        <origin xyz="0 0 0" rpy="1.57079632679 0 0"/>
         <geometry>
           <cylinder radius="${radius}" length="${width}"/>
@@ -38,7 +38,6 @@
       <parent link="${parent}"/>
       <child link="${name}"/>
-      <origin xyz="${x} ${y} ${z}" rpy="-1.57079632679 0 0"/>
-      <!-- Keep cylinder along link-Z and rotate the joint frame so wheel axle aligns with parent Y. -->
-      <axis xyz="0 0 1"/>
+      <origin xyz="${x} ${y} ${z}" rpy="0 0 0"/>
+      <axis xyz="0 1 0"/>
     </joint>
   </xacro:macro>
