Commit message: launch my robot in custom world

File: my_robot_description/urdf/komatsu.urdf.xacro (robot description, xacro)
@@ -127,5 +127,5 @@
     <parent link="rear_chassis"/>
     <child link="laser_frame"/>
-    <origin xyz="0.0 0.0 ${box_h + 0.3}" rpy="0 0 0"/> <!-- lidar 30 cm above the cabin -->
+    <origin xyz="0.0 0.0 1.2" rpy="0 0 0"/> <!-- Keep lidar lower so 2D scans see field obstacles -->
   </joint>
   <link name="imu_link"/>

File: my_robot_description/urdf/komatsu_gazebo.urdf.xacro (robot description, xacro)
@@ -110,5 +110,5 @@
             <!-- Output -->
             <publish_odom>true</publish_odom>
-            <publish_odom_tf>false</publish_odom_tf>
+            <publish_odom_tf>true</publish_odom_tf>
             <publish_wheel_tf>false</publish_wheel_tf>
             <odometry_frame>odom</odometry_frame>

Commit message: keep up lidar

File: my_robot_description/urdf/komatsu.urdf.xacro (robot description, xacro)
@@ -127,5 +127,5 @@
     <parent link="rear_chassis"/>
     <child link="laser_frame"/>
-    <origin xyz="0.0 0.0 1.2" rpy="0 0 0"/> <!-- Keep lidar lower so 2D scans see field obstacles -->
+      <origin xyz="0.0 0.0 ${box_h + 0.3}" rpy="0 0 0"/> <!-- lidar 30 cm above the cabin -->
   </joint>
   <link name="imu_link"/>

Commit message: fix shaking robot

File: my_robot_description/urdf/komatsu.urdf.xacro (robot description, xacro)
@@ -90,17 +90,14 @@
             o_rpy="0 0 0"/>
     </link>
-    <!-- articulation joints -->
-    <joint name="articulation_to_front" type="revolute">
+    <!-- articulation joints - TEMPORARILY FIXED FOR STABILITY, will be revolute with steering control -->
+    <joint name="articulation_to_front" type="fixed">
         <parent link="articulation_link"/>
         <child link="front_chassis"/>
-        <axis xyz="0 0 1"/>
-        <limit lower="-0.35" upper="0.35" effort="5000" velocity="0.196"/>
+        <origin xyz="0 0 0" rpy="0 0 0"/>
     </joint>
-    <joint name="articulation_to_rear" type="revolute">
+    <joint name="articulation_to_rear" type="fixed">
         <parent link="articulation_link"/>
         <child link="rear_chassis"/>
-        <axis xyz="0 0 1"/>
-        <limit lower="-0.35" upper="0.35" effort="5000" velocity="0.196"/>
-        <mimic joint="articulation_to_front" multiplier="-1"/>
+        <origin xyz="0 0 0" rpy="0 0 0"/>
     </joint>
   <!-- ===== Wheel macro ===== -->

File: my_robot_description/urdf/komatsu_gazebo.urdf.xacro (robot description, xacro)
@@ -134,3 +134,16 @@
         </plugin>
     </gazebo>
+    <!-- ===== Joint State Publisher Plugin ===== -->
+    <gazebo>
+        <plugin name="joint_state_publisher" filename="libgazebo_ros_joint_state_publisher.so">
+            <ros>
+                <namespace>/</namespace>
+            </ros>
+            <update_rate>50.0</update_rate>
+            <joint_name>rear_left_wheel_joint</joint_name>
+            <joint_name>rear_right_wheel_joint</joint_name>
+            <joint_name>front_left_wheel_joint</joint_name>
+            <joint_name>front_right_wheel_joint</joint_name>
+        </plugin>
+    </gazebo>
 </robot>

Commit message: use base link on gazebo

File: my_robot_description/urdf/komatsu.urdf.xacro (robot description, xacro)
@@ -25,18 +25,12 @@
     <xacro:property name="rbox_h" value="${H_height-F_clearance}"/>
     <xacro:property name="fbox_h" value="${H_height-F_clearance}"/>
-    <!-- base footprint -->
+    <!-- base link (physical root / articulation center reference) -->
+    <link name="base_link"/>
+    <!-- Ground-projected reference frame (no visual/collision/inertial) -->
     <link name="base_footprint"/>
-    <!-- base link (articulation center reference) -->
-    <link name="base_link">
-        <inertial>
-            <mass value="0.01"/>
-            <origin xyz="0 0 0" rpy="0 0 0"/>
-            <inertia ixx="0.001" ixy="0.0" ixz="0.0" iyy="0.001" iyz="0.0" izz="0.001"/>
-        </inertial>
-    </link>
     <joint name="base_footprint_joint" type="fixed">
-        <parent link="base_footprint"/>
-        <child link="base_link"/>
-        <origin xyz="0 0 ${F_clearance}" rpy="0 0 0"/>
+        <parent link="base_link"/>
+        <child link="base_footprint"/>
+        <origin xyz="0 0 ${-F_clearance}" rpy="0 0 0"/>
     </joint>
     <!-- articulation center -->

File: my_robot_description/urdf/komatsu_gazebo.urdf.xacro (robot description, xacro)
@@ -129,5 +129,5 @@
                 <remapping>odom:=ground_truth/odom</remapping>
             </ros>
-            <body_name>base_footprint</body_name>
+            <body_name>base_link</body_name>
             <frame_name>odom</frame_name>
             <update_rate>50.0</update_rate>

Commit message: update xacro for wheel joint z = 0

File: my_robot_description/urdf/komatsu.urdf.xacro (robot description, xacro)
@@ -7,30 +7,28 @@
     <material name="green"><color rgba="0.0 1.0 0.0 1.0"/></material>
     <material name="red"><color rgba="1.0 0.0 0.0 1.0"/></material>
-  <!-- ===== Dimensions ===== -->
-  <xacro:property name="A_len" value="8.350"/>
-  <xacro:property name="B_wheelbase" value="3.030"/>
-  <xacro:property name="D_width" value="2.765"/>
-  <xacro:property name="E_track" value="2.160"/>
-  <xacro:property name="F_clearance" value="0.455"/>
-  <xacro:property name="H_height" value="3.395"/>
-  <xacro:property name="X_len" value="2.660"/> <!-- axes to front and axes to rear -->
-  <xacro:property name="half_wb" value="${B_wheelbase/2.0}"/>
-  <xacro:property name="wheel_radius" value="0.80"/>
-  <xacro:property name="wheel_width" value="0.65"/>
-  <xacro:property name="wheel_y" value="${E_track/2.0}"/>
-  <xacro:property name="rear_box_len" value="${X_len + half_wb}"/>
-  <xacro:property name="front_box_len" value="${X_len + half_wb}"/>
-  <xacro:property name="box_w" value="${D_width-(2*wheel_width)}"/>
-  <xacro:property name="box_h" value="${H_height-F_clearance}"/>
-    <xacro:property name="rbox_h" value="${H_height-F_clearance}"/>
-    <xacro:property name="fbox_h" value="${H_height-F_clearance}"/>
-    <!-- base link (physical root / articulation center reference) -->
+    <!-- ===== Dimensions ===== -->
+    <xacro:property name="A_len" value="8.350"/>
+    <xacro:property name="B_wheelbase" value="3.030"/>
+    <xacro:property name="D_width" value="2.765"/>
+    <xacro:property name="E_track" value="2.160"/>
+    <xacro:property name="F_clearance" value="0.455"/>
+    <xacro:property name="H_height" value="3.395"/>
+    <xacro:property name="X_len" value="2.660"/> <!-- axes to front and axes to rear -->
+    <xacro:property name="half_wb" value="${B_wheelbase/2.0}"/>
+    <xacro:property name="wheel_radius" value="0.80"/>
+    <xacro:property name="wheel_width" value="0.65"/>
+    <xacro:property name="wheel_y" value="${E_track/2.0}"/>
+    <xacro:property name="rear_box_len" value="${X_len + half_wb}"/>
+    <xacro:property name="front_box_len" value="${X_len + half_wb}"/>
+    <xacro:property name="box_w" value="${D_width-(2*wheel_width)}"/>
+    <xacro:property name="box_h" value="${H_height-F_clearance}"/>
+    <!-- Ground frame -->
+    <link name="base_footprint"/>
+    <!-- Main robot reference at wheel axle / articulation height -->
     <link name="base_link"/>
-    <!-- Ground-projected reference frame (no visual/collision/inertial) -->
-    <link name="base_footprint"/>
-    <joint name="base_footprint_joint" type="fixed">
-        <parent link="base_link"/>
-        <child link="base_footprint"/>
-        <origin xyz="0 0 ${-F_clearance}" rpy="0 0 0"/>
+    <joint name="base_link_joint" type="fixed">
+        <parent link="base_footprint"/>
+        <child link="base_link"/>
+        <origin xyz="0 0 ${wheel_radius}" rpy="0 0 0"/>
     </joint>
     <!-- articulation center -->
@@ -45,44 +43,48 @@
         <parent link="base_link"/>
         <child link="articulation_link"/>
+        <origin xyz="0 0 0" rpy="0 0 0"/>
     </joint>
+    <!-- Body center relative to axle-height frame -->
+    <xacro:property name="body_center_z" value="${F_clearance + box_h/2.0 - wheel_radius}"/>
+    <xacro:property name="body_top_z" value="${body_center_z + box_h/2.0}"/>
     <!-- rear body -->
     <link name="rear_chassis">
         <visual>
-            <origin xyz="${-rear_box_len/2.0} 0 ${rbox_h/2.0}"/>
-            <geometry><box size="${rear_box_len} ${box_w} ${rbox_h}"/></geometry>
+            <origin xyz="${-rear_box_len/2.0} 0 ${body_center_z}"/>
+            <geometry><box size="${rear_box_len} ${box_w} ${box_h}"/></geometry>
             <material name="red"/>
         </visual>
         <collision>
-            <origin xyz="${-rear_box_len/2.0} 0 ${rbox_h/2.0}"/>
-            <geometry><box size="${rear_box_len} ${box_w} ${rbox_h}"/></geometry>
+            <origin xyz="${-rear_box_len/2.0} 0 ${body_center_z}"/>
+            <geometry><box size="${rear_box_len} ${box_w} ${box_h}"/></geometry>
         </collision>
         <xacro:box_inertia
-            m="500.0"
-            x="${rear_box_len}"
-            y="${box_w}"
-            z="${rbox_h}"
-            o_xyz="${-rear_box_len/2.0} 0 ${rbox_h/2.0}"
-            o_rpy="0 0 0"/>
+                m="500.0"
+                x="${rear_box_len}"
+                y="${box_w}"
+                z="${box_h}"
+                o_xyz="${-rear_box_len/2.0} 0 ${body_center_z}"
+                o_rpy="0 0 0"/>
     </link>
     <!-- front body -->
     <link name="front_chassis">
         <visual>
-            <origin xyz="${front_box_len/2.0} 0 ${fbox_h/2.0}"/>
-            <geometry><box size="${front_box_len} ${box_w} ${fbox_h}"/></geometry>
+            <origin xyz="${front_box_len/2.0} 0 ${body_center_z}"/>
+            <geometry><box size="${front_box_len} ${box_w} ${box_h}"/></geometry>
             <material name="green"/>
         </visual>
         <collision>
-            <origin xyz="${front_box_len/2.0} 0 ${fbox_h/2.0}"/>
-            <geometry><box size="${front_box_len} ${box_w} ${fbox_h}"/></geometry>
+            <origin xyz="${front_box_len/2.0} 0 ${body_center_z}"/>
+            <geometry><box size="${front_box_len} ${box_w} ${box_h}"/></geometry>
         </collision>
         <xacro:box_inertia
-            m="500.0"
-            x="${front_box_len}"
-            y="${box_w}"
-            z="${fbox_h}"
-            o_xyz="${front_box_len/2.0} 0 ${fbox_h/2.0}"
-            o_rpy="0 0 0"/>
+                m="500.0"
+                x="${front_box_len}"
+                y="${box_w}"
+                z="${box_h}"
+                o_xyz="${front_box_len/2.0} 0 ${body_center_z}"
+                o_rpy="0 0 0"/>
     </link>
-    <!-- articulation joints - TEMPORARILY FIXED FOR STABILITY, will be revolute with steering control -->
+    <!-- articulation joints - temporarily fixed for stability -->
     <joint name="articulation_to_front" type="fixed">
         <parent link="articulation_link"/>
@@ -95,34 +97,35 @@
         <origin xyz="0 0 0" rpy="0 0 0"/>
     </joint>
-  <!-- ===== Wheel macro ===== -->
-  <xacro:wheel name="rear_left_wheel"  parent="rear_chassis" x="${-half_wb}" y="${ wheel_y}" z="${wheel_radius - F_clearance}"/>
-  <xacro:wheel name="rear_right_wheel" parent="rear_chassis" x="${-half_wb}" y="${-wheel_y}" z="${wheel_radius - F_clearance}"/>
-  <xacro:wheel name="front_left_wheel"  parent="front_chassis" x="${ half_wb}" y="${ wheel_y}" z="${wheel_radius - F_clearance}"/>
-  <xacro:wheel name="front_right_wheel" parent="front_chassis" x="${ half_wb}" y="${-wheel_y}" z="${wheel_radius - F_clearance}"/>
-  <!-- ===== Navigation reference frames ===== -->
-  <link name="base_front"/>
-  <joint name="base_front_joint" type="fixed">
-    <parent link="front_chassis"/>
-    <child link="base_front"/>
-    <origin xyz="${half_wb} 0 0" rpy="0 0 0"/>
-  </joint>
-  <link name="base_rear"/>
-  <joint name="base_rear_joint" type="fixed">
-    <parent link="rear_chassis"/>
-    <child link="base_rear"/>
-    <origin xyz="${-half_wb} 0 0" rpy="0 0 0"/>
-  </joint>
-  <!-- ===== Sensors ===== -->
-  <link name="laser_frame"/>
-  <joint name="laser_joint" type="fixed">
-    <parent link="rear_chassis"/>
-    <child link="laser_frame"/>
-      <origin xyz="0.0 0.0 ${box_h + 0.3}" rpy="0 0 0"/> <!-- lidar 30 cm above the cabin -->
-  </joint>
-  <link name="imu_link"/>
-  <joint name="imu_joint" type="fixed">
-    <parent link="base_link"/>
-    <child link="imu_link"/>
-    <origin xyz="0 0 0" rpy="0 0 0"/>
-  </joint>
+    <!-- ===== Wheels ===== -->
+    <!-- Chassis link origins are at axle height, so wheel centers are z=0 relative to them -->
+    <xacro:wheel name="rear_left_wheel"  parent="rear_chassis"  x="${-half_wb}" y="${ wheel_y}" z="0.0" radius="${wheel_radius}" width="${wheel_width}"/>
+    <xacro:wheel name="rear_right_wheel" parent="rear_chassis"  x="${-half_wb}" y="${-wheel_y}" z="0.0" radius="${wheel_radius}" width="${wheel_width}"/>
+    <xacro:wheel name="front_left_wheel"  parent="front_chassis" x="${ half_wb}" y="${ wheel_y}" z="0.0" radius="${wheel_radius}" width="${wheel_width}"/>
+    <xacro:wheel name="front_right_wheel" parent="front_chassis" x="${ half_wb}" y="${-wheel_y}" z="0.0" radius="${wheel_radius}" width="${wheel_width}"/>
+    <!-- ===== Navigation reference frames ===== -->
+    <link name="base_front"/>
+    <joint name="base_front_joint" type="fixed">
+        <parent link="front_chassis"/>
+        <child link="base_front"/>
+        <origin xyz="${half_wb} 0 0" rpy="0 0 0"/>
+    </joint>
+    <link name="base_rear"/>
+    <joint name="base_rear_joint" type="fixed">
+        <parent link="rear_chassis"/>
+        <child link="base_rear"/>
+        <origin xyz="${-half_wb} 0 0" rpy="0 0 0"/>
+    </joint>
+    <!-- ===== Sensors ===== -->
+    <link name="laser_frame"/>
+    <joint name="laser_joint" type="fixed">
+        <parent link="rear_chassis"/>
+        <child link="laser_frame"/>
+        <origin xyz="0.0 0.0 ${body_top_z + 0.3}" rpy="0 0 0"/>
+    </joint>
+    <link name="imu_link"/>
+    <joint name="imu_joint" type="fixed">
+        <parent link="base_link"/>
+        <child link="imu_link"/>
+        <origin xyz="0 0 0" rpy="0 0 0"/>
+    </joint>
 </robot>
